File: PDB-FC.kicad_pcb (KiCad board)
At the start: 4 copper layers, 34.5 x 34.5 mm, 44 parts, among them J1 Conn_01x02, J10 Conn_01x02, J11 Conn_01x02, J12 Conn_01x02, J2 Conn_01x02, J3 Conn_01x02, J4 Conn_01x02, J5 Conn_01x02, J6 Conn_01x02, J7 Conn_01x02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

Commit message: add logo
Parts:
- added G***: LOGO, MyLogo:bit2byte_15m-x2mm, B.Cu at (146.8, 90.2)
